Commit message: find automatically the src folder

File: display_urdf/urdf/defects1.urdf (robot description, URDF)
Before this commit: robot robot_name, 2 links, 1 joints
Links:
- link defects: geometry visual mesh filename=file:///home/robotics/ros2_ws_git/src/display_urdf/stl/matt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 scale=0.001 0.001 0.001
