Commit message: changed name package urdf

File: display_with_rviz2/urdf/defects1.urdf (robot description, URDF)
Before this commit: robot robot_name, 2 links, 1 joints
Links:
- link defects: geometry visual mesh filename=file:///home/robotics/ros2_ws_git/src/display_with_rviz2/st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 scale=0.001 0.001 0.001

Commit message: feasible to work with no camera connected

File: display_with_rviz2/urdf/defects1.urdf (robot description, URDF)
Before this commit: robot robot_name, 2 links, 1 joints
Links:
- link defects: geometry visual mesh filename=file:///home/matteo/ros2_ws_git/src/display_with_rviz2/stl/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 scale=0.001 0.001 0.001
